Commit message: swaped filed to a different folder

File: bot_description/urdf/bot.xacro (robot description, xacro)
@@ -5,130 +5,167 @@
 <xacro:include filename="$(find bot_description)/urdf/bot.gazebo" />
 <link name="base_link">
-  <inertial>
-    <origin rpy="0 0 0" xyz="-0.273515310417399 0.0641923281592633 0.549094606768639"/>
-    <mass value="0.3413535466999629"/>
-    <inertia ixx="5.9e-05" ixy="-0.0" ixz="-0.0" iyy="0.000497" iyz="0.0" izz="0.000496"/>
-  </inertial>
-  <visual>
-    <origin rpy="0 0 0" xyz="0 0 0"/>
-    <geometry>
-      <mesh filename="package://bot_description/meshes/base_link.stl" scale="0.001 0.001 0.001"/>
-    </geometry>
-    <material name="silver"/>
-  </visual>
-  <collision>
-    <origin rpy="0 0 0" xyz="0 0 0"/>
-    <geometry>
-      <mesh filename="package://bot_description/meshes/base_link.stl" scale="0.001 0.001 0.001"/>
-    </geometry>
-  </collision>
+    <inertial>
+        <origin rpy="0 0 0" xyz="-0.273515310417399 0.0641923281592633 0.549094606768639"/>
+        <mass value="0.600"/>
+        <inertia ixx="5.9e-05" ixy="-0.0" ixz="-0.0" iyy="0.000497" iyz="0.0" izz="0.000496"/>
+    </inertial>
+    <visual>
+        <origin rpy="0 0 0" xyz="0 0 0"/>
+        <geometry>
+            <mesh filename="package://bot_description/meshes/base_link.stl" scale="0.001 0.001 0.001"/>
+        </geometry>
+        <material name="silver"/>
+    </visual>
+    <collision>
+        <origin rpy="0 0 0" xyz="0 0 0"/>
+        <geometry>
+            <mesh filename="package://bot_description/meshes/base_link.stl" scale="0.001 0.001 0.001"/>
+        </geometry>
+    </collision>
 </link>
 <link name="servo_arm_1_1_1">
-  <inertial>
-    <origin rpy="0 0 0" xyz="0.040123964751155816 2.284167705488005e-05 -0.13042234430764715"/>
-    <mass value="0.31691317622323045"/>
-    <inertia ixx="0.002875" ixy="0.0" ixz="-2.3e-05" iyy="0.002924" iyz="-0.0" izz="0.000106"/>
-  </inertial>
-  <visual>
-    <origin rpy="0 0 0" xyz="0.203153 -0.064192 -0.566678"/>
-    <geometry>
-      <mesh filename="package://bot_description/meshes/servo_arm_1_1_1.stl" scale="0.001 0.001 0.001"/>
-    </geometry>
-    <material name="silver"/>
-  </visual>
-  <collision>
-    <origin rpy="0 0 0" xyz="0.203153 -0.064192 -0.566678"/>
-    <geometry>
-      <mesh filename="package://bot_description/meshes/servo_arm_1_1_1.stl" scale="0.001 0.001 0.001"/>
-    </geometry>
-  </collision>
+    <inertial>
+        <origin rpy="0 0 0" xyz="0.040123964751155816 2.284167705488005e-05 -0.13042234430764715"/>
+        <mass value="0.330"/>
+        <inertia ixx="0.002875" ixy="0.0" ixz="-2.3e-05" iyy="0.002924" iyz="-0.0" izz="0.000106"/>
+    </inertial>
+    <visual>
+        <origin rpy="0 0 0" xyz="0.203153 -0.064192 -0.566678"/>
+        <geometry>
+            <mesh filename="package://bot_description/meshes/servo_arm_1_1_1.stl" scale="0.001 0.001 0.001"/>
+        </geometry>
+        <material name="silver"/>
+    </visual>
+    <collision>
+        <origin rpy="0 0 0" xyz="0.203153 -0.064192 -0.566678"/>
+        <geometry>
+            <mesh filename="package://bot_description/meshes/servo_arm_1_1_1.stl" scale="0.001 0.001 0.001"/>
+        </geometry>
+    </collision>
 </link>
 <link name="servo_arm_1_1_Mirror__1">
-  <inertial>
-    <origin rpy="0 0 0" xyz="-0.04012358502543206 2.284166630503459e-05 -0.13042234045956508"/>
-    <mass value="0.31691318435832444"/>
-    <inertia ixx="0.002875" ixy="-0.0" ixz="2.3e-05" iyy="0.002924" iyz="-0.0" izz="0.000106"/>
-  </inertial>
-  <visual>
-    <origin rpy="0 0 0" xyz="0.343878 -0.064192 -0.566678"/>
-    <geometry>
-      <mesh filename="package://bot_description/meshes/servo_arm_1_1_Mirror__1.stl" scale="0.001 0.001 0.001"/>
-    </geometry>
-    <material name="silver"/>
-  </visual>
-  <collision>
-    <origin rpy="0 0 0" xyz="0.343878 -0.064192 -0.566678"/>
-    <geometry>
-      <mesh filename="package://bot_description/meshes/servo_arm_1_1_Mirror__1.stl" scale="0.001 0.001 0.001"/>
-    </geometry>
-  </collision>
+    <inertial>
+        <origin rpy="0 0 0" xyz="-0.04012358502543206 2.284166630503459e-05 -0.13042234045956508"/>
+        <mass value="0.330"/>
+        <inertia ixx="0.002875" ixy="-0.0" ixz="2.3e-05" iyy="0.002924" iyz="-0.0" izz="0.000106"/>
+    </inertial>
+    <visual>
+        <origin rpy="0 0 0" xyz="0.343878 -0.064192 -0.566678"/>
+        <geometry>
+            <mesh filename="package://bot_description/meshes/servo_arm_1_1_Mirror__1.stl" scale="0.001 0.001 0.001"/>
+        </geometry>
+        <material name="silver"/>
+    </visual>
+    <collision>
+        <origin rpy="0 0 0" xyz="0.343878 -0.064192 -0.566678"/>
+        <geometry>
+            <mesh filename="package://bot_description/meshes/servo_arm_1_1_Mirror__1.stl" scale="0.001 0.001 0.001"/>
+        </geometry>
+    </collision>
 </link>
 <link name="dsnu-20-200-pps-a_03_1_1_1">
-  <inertial>
-    <origin rpy="0 0 0" xyz="0.019645702220741745 1.374704084221301e-05 -0.07233661753710188"/>
-    <mass value="0.3040090766287068"/>
-    <inertia ixx="0.006662" ixy="-0.0" ixz="-0.000264" iyy="0.006701" iyz="-0.0" izz="4.6e-05"/>
-  </inertial>
-  <visual>
-    <origin rpy="0 0 0" xyz="0.179003 -0.064193 -0.296678"/>
-    <geometry>
-      <mesh filename="package://bot_description/meshes/dsnu-20-200-pps-a_03_1_1_1.stl" scale="0.001 0.001 0.001"/>
-    </geometry>
-    <material name="silver"/>
-  </visual>
-  <collision>
-    <origin rpy="0 0 0" xyz="0.179003 -0.064193 -0.296678"/>
-    <geometry>
-      <mesh filename="package://bot_description/meshes/dsnu-20-200-pps-a_03_1_1_1.stl" scale="0.001 0.001 0.001"/>
-    </geometry>
-  </collision>
+    <inertial>
+        <origin rpy="0 0 0" xyz="0.019645702220741745 1.374704084221301e-05 0.09233661753710188"/>
+        <mass value="0.120"/>
+        <inertia ixx="0.006662" ixy="-0.0" ixz="-0.000264" iyy="0.006701" iyz="-0.0" izz="4.6e-05"/>
+    </inertial>
+    <visual>
+        <origin rpy="0 0 0" xyz="0.179003 -0.064193 -0.296678"/>
+        <geometry>
+            <mesh filename="package://bot_description/meshes/dsnu-20-200-pps-a_03_1_1_1.stl" scale="0.001 0.001 0.001"/>
+        </geometry>
+        <material name="silver"/>
+    </visual>
+    <collision>
+        <origin rpy="0 0 0" xyz="0.179003 -0.064193 -0.296678"/>
+        <geometry>
+            <mesh filename="package://bot_description/meshes/dsnu-20-200-pps-a_03_1_1_1.stl" scale="0.001 0.001 0.001"/>
+        </geometry>
+    </collision>
 </link>
 <link name="dsnu-20-200-pps-a_03_1_1_Mirror__1">
-  <inertial>
-    <origin rpy="0 0 0" xyz="-0.019645323075704824 1.374704085707612e-05 -0.07233661739654718"/>
-    <mass value="0.3040090763168277"/>
-    <inertia ixx="0.006662" ixy="0.0" ixz="0.000264" iyy="0.006701" iyz="-0.0" izz="4.6e-05"/>
-  </inertial>
-  <visual>
-    <origin rpy="0 0 0" xyz="0.368028 -0.064193 -0.296678"/>
-    <geometry>
-      <mesh filename="package://bot_description/meshes/dsnu-20-200-pps-a_03_1_1_Mirror__1.stl" scale="0.001 0.001 0.001"/>
-    </geometry>
-    <material name="silver"/>
-  </visual>
-  <collision>
-    <origin rpy="0 0 0" xyz="0.368028 -0.064193 -0.296678"/>
-    <geometry>
-      <mesh filename="package://bot_description/meshes/dsnu-20-200-pps-a_03_1_1_Mirror__1.stl" scale="0.001 0.001 0.001"/>
-    </geometry>
-  </collision>
+    <inertial>
+        <origin rpy="0 0 0" xyz="-0.019645323075704824 1.374704085707612e-05 0.09233661739654718"/>
+        <mass value="0.120"/>
+        <inertia ixx="0.006662" ixy="0.0" ixz="0.000264" iyy="0.006701" iyz="-0.0" izz="4.6e-05"/>
+    </inertial>
+    <visual>
+        <origin rpy="0 0 0" xyz="0.368028 -0.064193 -0.296678"/>
+        <geometry>
+            <mesh filename="package://bot_description/meshes/dsnu-20-200-pps-a_03_1_1_Mirror__1.stl" scale="0.001 0.001 0.001"/>
+        </geometry>
+        <material name="silver"/>
+    </visual>
+    <collision>
+        <origin rpy="0 0 0" xyz="0.368028 -0.064193 -0.296678"/>
+        <geometry>
+            <mesh filename="package://bot_description/meshes/dsnu-20-200-pps-a_03_1_1_Mirror__1.stl" scale="0.001 0.001 0.001"/>
+        </geometry>
+    </collision>
 </link>
-<joint name="Rev22" type="revolute">
-  <origin rpy="0 0 0" xyz="-0.203153 0.064192 0.566678"/>
-  <parent link="base_link"/>
-  <child link="servo_arm_1_1_1"/>
-  <axis xyz="1.0 0.0 0.0"/>
-  <limit effort="100" lower="-1.570796" upper="1.570796" velocity="100"/>
+<!-- Joints -->
+<joint name="RevR" type="revolute">
+    <origin rpy="-1.570796 0 0" xyz="-0.203153 0.064192 0.566678"/>
+    <parent link="base_link"/>
+    <child link="servo_arm_1_1_1"/>
+    <axis xyz="1.0 0.0 0.0"/>
+    <limit effort="100" lower="0" upper="3.14159" velocity="100"/>
 </joint>
-<joint name="Rev23" type="revolute">
-  <origin rpy="0 0 0" xyz="-0.343878 0.064192 0.566678"/>
-  <parent link="base_link"/>
-  <child link="servo_arm_1_1_Mirror__1"/>
-  <axis xyz="1.0 0.0 0.0"/>
-  <limit effort="100" lower="-1.570796" upper="1.570796" velocity="100"/>
+<joint name="RevL" type="revolute">
+    <origin rpy="-1.570796 0 0" xyz="-0.343878 0.064192 0.566678"/>
+    <parent link="base_link"/>
+    <child link="servo_arm_1_1_Mirror__1"/>
+    <axis xyz="1.0 0.0 0.0"/>
+    <limit effort="100" lower="0" upper="3.14159" velocity="100"/>
 </joint>
 <joint name="SliderR" type="prismatic">
-  <origin rpy="0 0 0" xyz="0.02415 1e-06 -0.27"/>
-  <parent link="servo_arm_1_1_1"/>
-  <child link="dsnu-20-200-pps-a_03_1_1_1"/>
-  <axis xyz="0.0 0.0 -1.0"/>
-  <limit effort="100" lower="0.0" upper="0.19" velocity="100"/>
+    <origin rpy="0 0 0" xyz="0.02415 1e-06 -0.27"/>
+    <parent link="servo_arm_1_1_1"/>
+    <child link="dsnu-20-200-pps-a_03_1_1_1"/>
+    <axis xyz="0.0 0.0 -1.0"/>
+    <limit effort="200" lower="0.0" upper="0.19" velocity="500"/>
+    <dynamics damping="50"/>
 </joint>
 <joint name="SliderL" type="prismatic">
-  <origin rpy="0 0 0" xyz="-0.02415 1e-06 -0.27"/>
-  <parent link="servo_arm_1_1_Mirror__1"/>
-  <child link="dsnu-20-200-pps-a_03_1_1_Mirror__1"/>
-  <axis xyz="0.0 0.0 -1.0"/>
-  <limit effort="100" lower="0.0" upper="0.19" velocity="100"/>
+    <origin rpy="0 0 0" xyz="-0.02415 1e-06 -0.27"/>
+    <parent link="servo_arm_1_1_Mirror__1"/>
+    <child link="dsnu-20-200-pps-a_03_1_1_Mirror__1"/>
+    <axis xyz="0.0 0.0 -1.0"/>
+    <limit effort="200" lower="0.0" upper="0.19" velocity="500"/>
+    <dynamics damping="50"/>
+</joint>
+<!-- Links to constrain to planar -->
+<link name="world"/>
+<link name="y_axis_link">
+    <collision>
+        <origin xyz="0 0 1" rpy="0 0 0"/>
+        <geometry>
+            <box size="0.01 0.01 0.01"/>
+        </geometry>
+    </collision>
+    <visual>
+        <origin xyz="0 0 1" rpy="0 0 0"/>
+        <geometry>
+            <box size="0.01 0.01 0.01"/>
+        </geometry>
+        <material name="silver"/>
+    </visual>
+    <inertial>
+        <origin xyz="0 0 1" rpy="0 0 0"/>
+        <mass value="0.01"/>
+        <inertia ixx="0.1" ixy="0.0" ixz="0.0" iyy="0.1" iyz="0.0" izz="0.1"/>
+    </inertial>
+</link>
+<joint name="y_direction" type="prismatic">
+    <parent link="world"/>
+    <child link="y_axis_link"/>
+    <axis xyz="0 1 0"/>
+    <limit effort="100" lower="-1.79769e+308" upper="1.79769e+308" velocity="100"/>
+</joint>
+<joint name="z_direction" type="prismatic">
+    <parent link="y_axis_link"/>
+    <child link="base_link"/>
+    <axis xyz="0 0 1"/>
+    <limit effort="100" lower="-1.79769e+308" upper="1.79769e+308" velocity="100"/>
 </joint>
 </robot>
