File: pcb/system/system.kicad_sch (KiCad schematic)
At the start: 10 parts, among them J1 Raspberry_Pi_4_GPIO, Q1 BS107A, Q2 BS107A, Q3 BS107A, Q4 BS107A

Commit message: pcb updated
Parts:
- added D? (x4): BZV55C3V3, Diode_SMD:D_MiniMELF, symbol Diode:BZV55C3V3
- added J?: Conn_01x05_Male, symbol Connector:Conn_01x05_Male
- added R? (x6): R, symbol pspice:R
- added Reg1: S13V30F5, symbol ze_symbols:S13V30F5
- gave numbers to parts that had none: 3
Connections:
- net GND: now also D?.2 (A)
- net +5V: now reaches R2.1
- net +5V: now also R1.1, R?.1, R?.1
- net at R1.2: now also D?.1 (K), R?.1
- net 3.3V: no longer names the net of J1.1 (Pin_1)
- net 3.3V: no longer J1.17 (Pin_17)
- net 5V: no longer names the net of J1.4 (Pin_4), J2.5 (Pin_5)
- net 5V: no longer J1.2 (Pin_2)
- net GPIO_0: no longer names the net of J1.27 (Pin_27)
- net GPIO_1: no longer names the net of J1.28 (Pin_28)
- net GPIO_10: no longer names the net of J1.19 (Pin_19)
- net GPIO_11: no longer names the net of J1.23 (Pin_23)
- net GPIO_12: no longer names the net of J1.32 (Pin_32), J3.1 (Pin_1)
- net GPIO_13: no longer names the net of J1.33 (Pin_33), J4.1 (Pin_1)
- net GPIO_14: no longer names the net of J1.8 (Pin_8)
- net GPIO_15: no longer names the net of J1.10 (Pin_10)
- net GPIO_16: no longer names the net of J1.36 (Pin_36)
- net GPIO_17: no longer names the net of J1.11 (Pin_11)
- net GPIO_18: no longer names the net of J1.12 (Pin_12)
- net GPIO_19: no longer names the net of J1.35 (Pin_35), Q1.2 (G)
- net GPIO_2: no longer names the net of J1.3 (Pin_3)
- net GPIO_20: no longer names the net of J1.38 (Pin_38)
- net GPIO_21: no longer names the net of J1.40 (Pin_40)
- net GPIO_22: no longer names the net of J1.15 (Pin_15)
- net GPIO_23: no longer names the net of J1.16 (Pin_16)
- net GPIO_24: no longer names the net of J1.18 (Pin_18)
- net GPIO_25: no longer names the net of J1.22 (Pin_22)
- net GPIO_26: no longer names the net of J1.37 (Pin_37), Q2.2 (G)
- net GPIO_27: no longer names the net of J1.13 (Pin_13)
- net GPIO_3: no longer names the net of J1.5 (Pin_5)
- net GPIO_4: no longer names the net of J1.7 (Pin_7)
- net GPIO_5: no longer names the net of J1.29 (Pin_29), Q4.2 (G)
- net GPIO_6: no longer names the net of J1.31 (Pin_31), Q3.2 (G)
- net GPIO_7: no longer names the net of J1.26 (Pin_26)
- net GPIO_8: no longer names the net of J1.24 (Pin_24)
- net GPIO_9: no longer names the net of J1.21 (Pin_21)
- removed net Ground: J1.14 (Pin_14), J1.20 (Pin_20), J1.25 (Pin_25), J1.30 (Pin_30), J1.34 (Pin_34), J1.39 (Pin_39), J1.6 (Pin_6), J1.9 (Pin_9), J2.4 (Pin_4)
- new net: J?.1 (Pin_1), Reg1.1 (EN)
- new net: J?.2 (Pin_2), Reg1.2 (V_in)
- new net: J?.3 (Pin_3), Reg1.3 (GND)
- new net: J?.4 (Pin_4), Reg1.4 (GND)
- new net: J?.5 (Pin_5), Reg1.5 (V_out)
- new net: J1.6 (Pin_6), J2.4 (Pin_4)
Other:
- note added: "3.3V"
- note added: "5V"
- note added: "Enable"
- note added: "GPIO_0"
- note added: "GPIO_1"
- note added: "GPIO_10"
- note added: "GPIO_11"
- note added: "GPIO_12"
- note added: "GPIO_13"
- note added: "GPIO_14"
- note added: "GPIO_15"
- note added: "GPIO_16"
- note added: "GPIO_17"
- note added: "GPIO_18"
- note added: "GPIO_19"
- note added: "GPIO_2"
- note added: "GPIO_20"
- note added: "GPIO_21"
- note added: "GPIO_22"
- note added: "GPIO_23"
- note added: "GPIO_24"
- note added: "GPIO_25"
- note added: "GPIO_26"
- note added: "GPIO_27"
- note added: "GPIO_3"
- note added: "GPIO_4"
- note added: "GPIO_5"
- note added: "GPIO_6"
- note added: "GPIO_7"
- note added: "GPIO_8"
- note added: "GPIO_9"
- note added: "Ground"
- note added: "V_in"
- note added: "V_out"
- moved on the sheet: R1, R2

Commit message: updated pcb
Parts:
- removed J2: 5V_Regulator_Female, symbol Connector:Conn_01x05_Female
- removed J?: Conn_01x05_Male, symbol Connector:Conn_01x05_Male
- added J? (x2): Screw_Terminal_01x02, symbol Connector:Screw_Terminal_01x02
- added SW?: SW_Push, symbol Switch:SW_Push
- added U?: Teensy4.0, symbol teensy:Teensy4.0
Connections:
- net +8V: now also Reg1.2 (V_in)
- net GND: now also D?.2 (A), D?.2 (A), D?.2 (A), Reg1.3 (GND)
- net at R?.2: now also D?.1 (K), R?.2, U?.10 (8_TX2_IN1)
- net at Reg1.4 (GND): now also J1.6 (Pin_6)
- net at Reg1.5 (V_out): now also J1.4 (Pin_4)
- net at R?.2: now also D?.1 (K), R?.2, U?.11 (9_OUT1C)
- net Encoder_2_B: now reaches R?.1
- net Encoder_2_B: now also R?.1, J?.1 (Pin_1), J?.1 (Pin_1)
- net at R?.2: now also D?.1 (K), R2.2, U?.8 (6_OUT1D)
- net at D?.1 (K), R1.2: now also R?.2, U?.7 (5_IN2); no longer R?.1
- net Encoder_2_A: now reaches R?.1
- net Encoder_2_A: now also J?.2 (Pin_2)
- net +5V: no longer names the net of R1.1, R2.1, R?.1, R?.1
- net +5V: now also SW?.1, U?.33 (VIN)
- new net: SW?.2, U?.14 (12_MISO_MQSL)
- new net Encoder_1_A: J?.2 (Pin_2), R?.1
- no-connect marks 1 -> 40
Other:
- note removed: "Enable"
- note removed: "V_in"
- note removed: "V_out"
- moved on the sheet: D?, R1, R2, R?, Reg1

Commit message: as
Parts:
- added J6: Screw_Terminal_01x02, TerminalBlock_4Ucon:TerminalBlock_4Ucon_1x02_P3.50mm_Vertical, symbol Connector:Screw_Terminal_01x02
- added Q5, Q6: IRF520, Package_TO_SOT_THT:TO-92L_Inline, symbol ze_symbols:IRF520
- added SW1: SW_SPST, Button_Switch_SMD:SW_DIP_SPSTx01_Slide_6.7x4.1mm_W6.73mm_P2.54mm_LowProfile_JPin, symbol Switch:SW_SPST
- added Sol1, Sol2, Sol3, Sol4: Solenoid, Connector_PinSocket_2.54mm:PinSocket_1x03_P2.54mm_Vertical, symbol ze_symbols:Solenoid
- D1, D2, D3, D4: renamed from D?; value BZV55C3V3 -> 1N746A; footprint Diode_SMD:D_MiniMELF -> Diode_THT:D_DO-35_SOD27_P7.62mm_Horizontal
- J1: footprint (none) -> Connector_PinSocket_2.54mm:PinSocket_2x20_P2.54mm_Vertical
- J2, J5: renamed from J?; footprint (none) -> TerminalBlock_4Ucon:TerminalBlock_4Ucon_1x02_P3.50mm_Vertical
- J3, J4: footprint (none) -> Connector_PinHeader_2.54mm:PinHeader_1x03_P2.54mm_Vertical
- Q1, Q2, Q3, Q4: footprint Package_TO_SOT_THT:TO-92_Inline -> Package_TO_SOT_THT:TO-92L_Inline
- R1, R2: value R -> 1.2k; footprint (none) -> Resistor_THT:R_Axial_DIN0204_L3.6mm_D1.6mm_P5.08mm_Horizontal
- R3, R4, R6, R8: renamed from R?; value R -> 110; footprint (none) -> Resistor_THT:R_Axial_DIN0204_L3.6mm_D1.6mm_P5.08mm_Horizontal
- R5, R7: renamed from R?; value R -> 1.2k; footprint (none) -> Resistor_THT:R_Axial_DIN0204_L3.6mm_D1.6mm_P5.08mm_Horizontal
- Reg1: footprint (none) -> Connector_PinSocket_2.54mm:PinSocket_1x05_P2.54mm_Vertical
- SW2: renamed from SW?; footprint (none) -> Button_Switch_THT:SW_PUSH_6mm
- U1: renamed from U?; footprint (none) -> teensy_library-master:Teensy40
Connections:
- net +8V: now also Q5.2 (D), Q6.2 (D)
- net Encoder_1_A: now also J2.1 (Pin_1); no longer J2.2 (Pin_2)
- net Encoder_2_B: no longer J2.1 (Pin_1), R4.1
- net GND: now also J3.3 (Pin_3), J4.3 (Pin_3), U1.1 (GND), U1.32 (GND)
- net at D4.1 (K), R7.2, R8.2: now also U1.11 (9_OUT1C); no longer U1.10 (8_TX2_IN1)
- net at D3.1 (K), R5.2, R6.2: now also U1.10 (8_TX2_IN1); no longer U1.11 (9_OUT1C)
- net at Q4.1 (D): now also Sol3.1
- net GPIO_5: now reaches J1.29 (Pin_29), Q4.2 (G)
- net at U1.22 (15_A1_RX3_SPDIF_IN): now also D2.1 (K), R2.2, R4.2
- net at U1.23 (16_A2_RX4_SCL1): now also D1.1 (K), R1.2, R3.2
- net Servo_Left: now reaches U1.29 (22_A8_CTX1)
- net Servo_Left: now also J6.2 (Pin_2)
- net Servo_Right: now reaches U1.30 (23_A9_CRX1_MCLK1)
- net Servo_Right: now also J6.1 (Pin_1)
- net at Q1.1 (D): now also Sol4.1
- net GPIO_19: now reaches J1.35 (Pin_35), Q1.2 (G)
- net 3.3V: now reaches J1.1 (Pin_1)
- net 3.3V: now also J1.17 (Pin_17), SW1.1 (A)
- net GPIO_15: now reaches J1.10 (Pin_10)
- net GPIO_17: now reaches J1.11 (Pin_11)
- net GPIO_18: now reaches J1.12 (Pin_12)
- net GPIO_27: now reaches J1.13 (Pin_13)
- net Ground: now reaches J1.14 (Pin_14)
- net Ground: now also J1.20 (Pin_20), J1.25 (Pin_25), J1.30 (Pin_30), J1.34 (Pin_34), J1.39 (Pin_39), J1.6 (Pin_6), J1.9 (Pin_9), Reg1.4 (GND)
- net GPIO_22: now reaches J1.15 (Pin_15)
- net GPIO_23: now reaches J1.16 (Pin_16)
- net GPIO_24: now reaches J1.18 (Pin_18)
- net GPIO_10: now reaches J1.19 (Pin_19)
- net 5V: now reaches J1.2 (Pin_2)
- net 5V: now also J1.4 (Pin_4), Reg1.5 (V_out)
- net GPIO_9: now reaches J1.21 (Pin_21)
- net GPIO_25: now reaches J1.22 (Pin_22)
- net GPIO_11: now reaches J1.23 (Pin_23)
- net GPIO_8: now reaches J1.24 (Pin_24)
- net GPIO_7: now reaches J1.26 (Pin_26)
- net GPIO_0: now reaches J1.27 (Pin_27)
- net GPIO_1: now reaches J1.28 (Pin_28)
- net GPIO_2: now reaches J1.3 (Pin_3)
- net GPIO_6: now reaches J1.31 (Pin_31), Q3.2 (G)
- net GPIO_12: now reaches J1.32 (Pin_32), J3.1 (Pin_1)
- net GPIO_13: now reaches J1.33 (Pin_33), J4.1 (Pin_1)
- net GPIO_16: now reaches J1.36 (Pin_36)
- net GPIO_26: now reaches J1.37 (Pin_37), Q2.2 (G)
- net GPIO_20: now reaches J1.38 (Pin_38)
- net GPIO_21: now reaches J1.40 (Pin_40)
- net GPIO_3: now reaches J1.5 (Pin_5)
- net GPIO_4: now reaches J1.7 (Pin_7)
- net GPIO_14: now reaches J1.8 (Pin_8)
- net at J4.2 (Pin_2): now also Q6.3 (S)
- net at J3.2 (Pin_2): now also Q5.3 (S)
- net at Q2.1 (D): now also Sol1.1
- net at Q3.1 (D): now also Sol2.1
- new net: Q5.1 (G), Q6.1 (G), SW1.2 (B)
- new net +24V: Sol1.2, Sol2.2, Sol3.2, Sol4.2
- new net Encoder_1_B: J2.2 (Pin_2), R4.1
- now unconnected: U1.7 (5_IN2), U1.8 (6_OUT1D)
- no-connect marks 40 -> 76
Other:
- note removed: "3.3V"
- note removed: "5V"
- note removed: "GPIO_0"
- note removed: "GPIO_1"
- note removed: "GPIO_10"
- note removed: "GPIO_11"
- note removed: "GPIO_12"
- note removed: "GPIO_13"
- note removed: "GPIO_14"
- note removed: "GPIO_15"
- note removed: "GPIO_16"
- note removed: "GPIO_17"
- note removed: "GPIO_18"
- note removed: "GPIO_19"
- note removed: "GPIO_2"
- note removed: "GPIO_20"
- note removed: "GPIO_21"
- note removed: "GPIO_22"
- note removed: "GPIO_23"
- note removed: "GPIO_24"
- note removed: "GPIO_25"
- note removed: "GPIO_26"
- note removed: "GPIO_27"
- note removed: "GPIO_3"
- note removed: "GPIO_4"
- note removed: "GPIO_5"
- note removed: "GPIO_6"
- note removed: "GPIO_7"
- note removed: "GPIO_8"
- note removed: "GPIO_9"
- note removed: "Ground"
- moved on the sheet: D1, D2, D3, D4, J2, J3, J5, Q1, R1, R2, R3, R4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

Commit message: copium
Parts:
- added J7: Screw_Terminal_01x02, TerminalBlock_4Ucon:TerminalBlock_4Ucon_1x02_P3.50mm_Vertical, symbol Connector:Screw_Terminal_01x02
- Q5, Q6: footprint Package_TO_SOT_THT:TO-92L_Inline -> Package_TO_SOT_THT:TO-92L_HandSolder
- SW1: footprint Button_Switch_SMD:SW_DIP_SPSTx01_Slide_6.7x4.1mm_W6.73mm_P2.54mm_LowProfile_JPin -> Button_Switch_THT:SW_CuK_JS202011CQN_DPDT_Straight
- SW2: footprint Button_Switch_THT:SW_PUSH_6mm -> Button_Switch_THT:SW_PUSH_6mm_H4.3mm
- Sol1, Sol2, Sol3, Sol4: footprint Connector_PinSocket_2.54mm:PinSocket_1x03_P2.54mm_Vertical -> Connector_PinSocket_2.54mm:PinSocket_1x02_P2.54mm_Vertical
Connections:
- net Ground is gone; now on net GND: J1.14 (Pin_14), J1.20 (Pin_20), J1.25 (Pin_25), J1.30 (Pin_30), J1.34 (Pin_34), J1.39 (Pin_39), J1.6 (Pin_6), J1.9 (Pin_9), Reg1.4 (GND)
- net +8V: now also J7.1 (Pin_1)
- net Encoder_1_A: now also J2.2 (Pin_2); no longer J2.1 (Pin_1)
- net Encoder_1_B: now also J2.1 (Pin_1); no longer J2.2 (Pin_2)
- net GND: now also J7.2 (Pin_2)
- net at R1.1, R2.1, R5.1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: no longer SW2.1
- net at U1.13 (11_MOSI_CTX1): now also SW2.1
- net at D2.1 (K), R2.2, R4.2: now also U1.8 (6_OUT1D); no longer U1.22 (15_A1_RX3_SPDIF_IN)
- net at D1.1 (K), R1.2, R3.2: now also U1.7 (5_IN2); no longer U1.23 (16_A2_RX4_SCL1)
- no-connect marks 76 -> 75
Other:
- moved on the sheet: J2, J5, SW2

Commit message: i think the pcb is done
Parts:
- Sol1, Sol2, Sol3, Sol4: footprint Connector_PinSocket_2.54mm:PinSocket_1x02_P2.54mm_Vertical -> Connector_PinSocket_2.54mm:PinSocket_1x01_P2.54mm_Vertical
Connections:
- removed net +24V: Sol1.2, Sol2.2, Sol3.2, Sol4.2
Changed lines of the file:
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@@
       (effects (font (size 1.27 1.27)) (justify left))
     )
-    (property "Footprint" "Connector_PinSocket_2.54mm:PinSocket_1x02_P2.54mm_Vertical" (id 2) (at 116.84 165.1 0)
+    (property "Footprint" "Connector_PinSocket_2.54mm:PinSocket_1x01_P2.54mm_Vertical" (id 2) (at 116.84 165.1 0)
       (effects (font (size 1.27 1.27)) hide)
     )
@@
     )
     (pin "1")
-    (pin "2")
   )
   (symbol (lib_id "pspice:R") (at 233.68 30.48 0) (unit 1)
@@
     (pin "2")
   )
-  (symbol (lib_id "ze_symbols:Solenoid") (at 116.84 151.13 0) (unit 1)
+  (symbol (lib_name "Solenoid_3") (lib_id "ze_symbols:Solenoid") (at 116.84 151.13 0) (unit 1)
     (in_bom yes) (on_board yes) (fields_autoplaced)
     (property "Reference" "Sol3" (id 0) (at 123.19 158.7499 0)
@@
       (effects (font (size 1.27 1.27)) (justify left))
     )
-    (property "Footprint" "Connector_PinSocket_2.54mm:PinSocket_1x02_P2.54mm_Vertical" (id 2) (at 116.84 151.13 0)
+    (property "Footprint" "Connector_PinSocket_2.54mm:PinSocket_1x01_P2.54mm_Vertical" (id 2) (at 116.84 151.13 0)
       (effects (font (size 1.27 1.27)) hide)
     )
@@
     )
     (pin "1")
-    (pin "2")
   )
   (symbol (lib_id "power:GND") (at 87.63 140.97 0) (unit 1)
@@
     (pin "3")
   )
-  (symbol (lib_id "ze_symbols:Solenoid") (at 116.84 135.89 0) (unit 1)
+  (symbol (lib_name "Solenoid_2") (lib_id "ze_symbols:Solenoid") (at 116.84 135.89 0) (unit 1)
     (in_bom yes) (on_board yes) (fields_autoplaced)
     (property "Reference" "Sol2" (id 0) (at 123.19 143.5099 0)
@@
       (effects (font (size 1.27 1.27)) (justify left))
     )
-    (property "Footprint" "Connector_PinSocket_2.54mm:PinSocket_1x02_P2.54mm_Vertical" (id 2) (at 116.84 135.89 0)
+    (property "Footprint" "Connector_PinSocket_2.54mm:PinSocket_1x01_P2.54mm_Vertical" (id 2) (at 116.84 135.89 0)
       (effects (font (size 1.27 1.27)) hide)
     )
@@
     )
     (pin "1")
-    (pin "2")
   )
   (symbol (lib_id "Switch:SW_Push") (at 157.48 114.3 270) (unit 1)
@@
     (pin "2")
   )
-  (symbol (lib_id "ze_symbols:Solenoid") (at 116.84 120.65 0) (unit 1)
+  (symbol (lib_name "Solenoid_1") (lib_id "ze_symbols:Solenoid") (at 116.84 120.65 0) (unit 1)
     (in_bom yes) (on_board yes) (fields_autoplaced)
     (property "Reference" "Sol1" (id 0) (at 123.19 128.2699 0)
@@
       (effects (font (size 1.27 1.27)) (justify left))
     )
-    (property "Footprint" "Connector_PinSocket_2.54mm:PinSocket_1x02_P2.54mm_Vertical" (id 2) (at 116.84 120.65 0)
+    (property "Footprint" "Connector_PinSocket_2.54mm:PinSocket_1x01_P2.54mm_Vertical" (id 2) (at 116.84 120.65 0)
       (effects (font (size 1.27 1.27)) hide)
     )
@@
     )
     (pin "1")
-    (pin "2")
   )
   (symbol (lib_id "pspice:R") (at 242.57 43.18 180) (unit 1)
@@
     (pin "1")
     (pin "2")
-  )
-  (symbol (lib_id "power:+24V") (at 111.76 175.26 90) (unit 1)
-    (in_bom yes) (on_board yes) (fields_autoplaced)
-    (property "Reference" "#PWR08" (id 0) (at 115.57 175.26 0)
-      (effects (font (size 1.27 1.27)) hide)
-    )
-    (property "Value" "+24V" (id 1) (at 107.95 175.2599 90)
-      (effects (font (size 1.27 1.27)) (justify left))
-    )
-    (property "Footprint" "" (id 2) (at 111.76 175.26 0)
-      (effects (font (size 1.27 1.27)) hide)
-    )
-    (property "Datasheet" "" (id 3) (at 111.76 175.26 0)
-      (effects (font (size 1.27 1.27)) hide)
-    )
-    (pin "1")
   )
   (symbol (lib_id "Connector:Screw_Terminal_01x02") (at 180.34 73.66 270) (unit 1)
@@
     (pin "1")
   )
-  (symbol (lib_id "power:+24V") (at 111.76 161.29 90) (unit 1)
-    (in_bom yes) (on_board yes) (fields_autoplaced)
-    (property "Reference" "#PWR07" (id 0) (at 115.57 161.29 0)
-      (effects (font (size 1.27 1.27)) hide)
-    )
-    (property "Value" "+24V" (id 1) (at 107.95 161.2899 90)
-      (effects (font (size 1.27 1.27)) (justify left))
-    )
-    (property "Footprint" "" (id 2) (at 111.76 161.29 0)
-      (effects (font (size 1.27 1.27)) hide)
-    )
-    (property "Datasheet" "" (id 3) (at 111.76 161.29 0)
-      (effects (font (size 1.27 1.27)) hide)
-    )
-    (pin "1")
-  )
-  (symbol (lib_id "power:+24V") (at 111.76 130.81 90) (unit 1)
-    (in_bom yes) (on_board yes) (fields_autoplaced)
-    (property "Reference" "#PWR05" (id 0) (at 115.57 130.81 0)
-      (effects (font (size 1.27 1.27)) hide)
-    )
-    (property "Value" "+24V" (id 1) (at 107.95 130.8099 90)
-      (effects (font (size 1.27 1.27)) (justify left))
-    )
-    (property "Footprint" "" (id 2) (at 111.76 130.81 0)
-      (effects (font (size 1.27 1.27)) hide)
-    )
-    (property "Datasheet" "" (id 3) (at 111.76 130.81 0)
-      (effects (font (size 1.27 1.27)) hide)
-    )
-    (pin "1")
-  )
-  (symbol (lib_id "power:+24V") (at 111.76 146.05 90) (unit 1)
-    (in_bom yes) (on_board yes) (fields_autoplaced)
-    (property "Reference" "#PWR06" (id 0) (at 115.57 146.05 0)
-      (effects (font (size 1.27 1.27)) hide)
-    )
-    (property "Value" "+24V" (id 1) (at 107.95 146.0499 90)
-      (effects (font (size 1.27 1.27)) (justify left))
-    )
-    (property "Footprint" "" (id 2) (at 111.76 146.05 0)
-      (effects (font (size 1.27 1.27)) hide)
-    )
-    (property "Datasheet" "" (id 3) (at 111.76 146.05 0)
-      (effects (font (size 1.27 1.27)) hide)
-    )
-    (pin "1")
-  )
   (symbol (lib_id "Connector:Screw_Terminal_01x02") (at 267.97 152.4 0) (unit 1)
     (in_bom yes) (on_board yes)
@@
       (reference "#PWR04") (unit 1) (value "GND") (footprint "")
     )
-    (path "/ec5237ce-d09a-43ef-a2f2-1609403e37ee"
-      (reference "#PWR05") (unit 1) (value "+24V") (footprint "")
-    )
-    (path "/ecaf6818-957a-4be9-93f5-6be93f2dff95"
-      (reference "#PWR06") (unit 1) (value "+24V") (footprint "")
-    )
-    (path "/e79be0c1-58d6-4b39-9b88-a8f6ac7ed6ae"
-      (reference "#PWR07") (unit 1) (value "+24V") (footprint "")
-    )
-    (path "/e336694c-16bc-493f-8c28-33fea2950cc8"
-      (reference "#PWR08") (unit 1) (value "+24V") (footprint "")
-    )
     (path "/c92fc722-ab94-42ac-8bb8-afc9da9f282c"
       (reference "#PWR09") (unit 1) (value "+8V6") (footprint "")
@@
     )
     (path "/9e3f26de-6b94-449f-b208-395648f613f9"
-      (reference "Sol1") (unit 1) (value "Solenoid") (footprint "Connector_PinSocket_2.54mm:PinSocket_1x02_P2.54mm_Vertical")
+      (reference "Sol1") (unit 1) (value "Solenoid") (footprint "Connector_PinSocket_2.54mm:PinSocket_1x01_P2.54mm_Vertical")
     )
     (path "/854bbd50-f4c3-43eb-9ff0-f20f68236d03"
-      (reference "Sol2") (unit 1) (value "Solenoid") (footprint "Connector_PinSocket_2.54mm:PinSocket_1x02_P2.54mm_Vertical")
+      (reference "Sol2") (unit 1) (value "Solenoid") (footprint "Connector_PinSocket_2.54mm:PinSocket_1x01_P2.54mm_Vertical")
     )
     (path "/635f602d-279b-468b-b0ca-2c4c49b6bbb2"
-      (reference "Sol3") (unit 1) (value "Solenoid") (footprint "Connector_PinSocket_2.54mm:PinSocket_1x02_P2.54mm_Vertical")
+      (reference "Sol3") (unit 1) (value "Solenoid") (footprint "Connector_PinSocket_2.54mm:PinSocket_1x01_P2.54mm_Vertical")
     )
     (path "/049d0226-c438-4f0e-8b83-9519d7d793ac"
-      (reference "Sol4") (unit 1) (value "Solenoid") (footprint "Connector_PinSocket_2.54mm:PinSocket_1x02_P2.54mm_Vertical")
+      (reference "Sol4") (unit 1) (value "Solenoid") (footprint "Connector_PinSocket_2.54mm:PinSocket_1x01_P2.54mm_Vertical")
     )
     (path "/4bf7c002-0e81-46f3-ad53-36186ead0aae"

Commit message: awe
Parts:
- added C1, C2: 22pF, Capacitor_THT:CP_Radial_Tantal_D4.5mm_P2.50mm, symbol pspice:CAP
- added J10, J9: Conn_02x08_Odd_Even, Connector_PinHeader_2.54mm:PinHeader_2x08_P2.54mm_Vertical, symbol Connector_Generic:Conn_02x08_Odd_Even
- added J11, J12: Conn_02x04_Odd_Even, Connector_PinHeader_2.54mm:PinHeader_2x04_P2.54mm_Vertical, symbol Connector_Generic:Conn_02x04_Odd_Even
- added J8: USB_A, Connector_USB:USB_A_Molex_105057_Vertical, symbol Connector:USB_A
- J1: footprint Connector_PinSocket_2.54mm:PinSocket_2x20_P2.54mm_Vertical -> Connector_PinHeader_2.54mm:PinHeader_2x20_P2.54mm_Vertical
- R1, R2, R5, R7: value 1.2k -> 1.2kΩ
- R3, R4, R6, R8: value 110 -> 110Ω
Connections:
- net 5V: no longer Reg1.5 (V_out)
- net GND: now also C1.2, C2.2, J8.4 (GND), J8.5 (Shield); no longer J1.14 (Pin_14), J1.20 (Pin_20), J1.25 (Pin_25), J1.30 (Pin_30), J1.34 (Pin_34), J1.39 (Pin_39), J1.6 (Pin_6), J1.9 (Pin_9)
- new net: C1.1, J8.2 (D-)
- new net: C2.1, J8.3 (D+)
- new net: J8.1 (VBUS), Reg1.5 (V_out)
- new net Ground: J1.14 (Pin_14), J1.20 (Pin_20), J1.25 (Pin_25), J1.30 (Pin_30), J1.34 (Pin_34), J1.39 (Pin_39), J1.6 (Pin_6), J1.9 (Pin_9)
- no-connect marks 75 -> 123
Other:
- moved on the sheet: Reg1

Commit message: thicker pcb traces
Parts:
- Q1, Q2, Q3, Q4: footprint Package_TO_SOT_THT:TO-92L_Inline -> Package_TO_SOT_THT:TO-92L_HandSolder
Changed lines of the file:
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@@
       (effects (font (size 1.27 1.27)) (justify left))
     )
-    (property "Footprint" "Package_TO_SOT_THT:TO-92L_Inline" (id 2) (at 90.17 156.845 0)
+    (property "Footprint" "Package_TO_SOT_THT:TO-92L_HandSolder" (id 2) (at 90.17 156.845 0)
       (effects (font (size 1.27 1.27) italic) (justify left) hide)
     )
@@
       (effects (font (size 1.27 1.27)) (justify left))
     )
-    (property "Footprint" "Package_TO_SOT_THT:TO-92L_Inline" (id 2) (at 50.8 155.575 0)
+    (property "Footprint" "Package_TO_SOT_THT:TO-92L_HandSolder" (id 2) (at 50.8 155.575 0)
       (effects (font (size 1.27 1.27) italic) (justify left) hide)
     )
@@
       (effects (font (size 1.27 1.27)) (justify left))
     )
-    (property "Footprint" "Package_TO_SOT_THT:TO-92L_Inline" (id 2) (at 62.23 137.795 0)
+    (property "Footprint" "Package_TO_SOT_THT:TO-92L_HandSolder" (id 2) (at 62.23 137.795 0)
       (effects (font (size 1.27 1.27) italic) (justify left) hide)
     )
@@
       (effects (font (size 1.27 1.27)) (justify left))
     )
-    (property "Footprint" "Package_TO_SOT_THT:TO-92L_Inline" (id 2) (at 90.17 137.795 0)
+    (property "Footprint" "Package_TO_SOT_THT:TO-92L_HandSolder" (id 2) (at 90.17 137.795 0)
       (effects (font (size 1.27 1.27) italic) (justify left) hide)
     )
@@
     )
     (path "/55b10beb-e630-475c-9ad7-7bfe00c4633e"
-      (reference "Q1") (unit 1) (value "BS107A") (footprint "Package_TO_SOT_THT:TO-92L_Inline")
+      (reference "Q1") (unit 1) (value "BS107A") (footprint "Package_TO_SOT_THT:TO-92L_HandSolder")
     )
     (path "/8c0cb532-1927-4285-b61a-2ee422d00156"
-      (reference "Q2") (unit 1) (value "BS107A") (footprint "Package_TO_SOT_THT:TO-92L_Inline")
+      (reference "Q2") (unit 1) (value "BS107A") (footprint "Package_TO_SOT_THT:TO-92L_HandSolder")
     )
     (path "/91eb6509-b3ff-427a-a767-5967de802698"
-      (reference "Q3") (unit 1) (value "BS107A") (footprint "Package_TO_SOT_THT:TO-92L_Inline")
+      (reference "Q3") (unit 1) (value "BS107A") (footprint "Package_TO_SOT_THT:TO-92L_HandSolder")
     )
     (path "/46f7f8c4-48a1-4c78-b885-23f0e351257a"
-      (reference "Q4") (unit 1) (value "BS107A") (footprint "Package_TO_SOT_THT:TO-92L_Inline")
+      (reference "Q4") (unit 1) (value "BS107A") (footprint "Package_TO_SOT_THT:TO-92L_HandSolder")
     )
     (path "/791fbfac-5281-4b93-9ad9-a5aba5135fdc"
