File: pcb/system/system.kicad_sch (KiCad schematic)
At the start: 40 parts, among them J1 Raspberry_Pi_4_GPIO, J10 Conn_02x08_Odd_Even, J11 Conn_02x04_Odd_Even, J12 Conn_02x04_Odd_Even, J2 Screw_Terminal_01x02, J3 Servo_1_Header, J4 Servo_2_Header, J5 Screw_Terminal_01x02, J6 Screw_Terminal_01x02, J7 Screw_Terminal_01x02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

Commit message: just making sure everything is pushed
Parts:
- removed J7: Screw_Terminal_01x02, TerminalBlock_4Ucon:TerminalBlock_4Ucon_1x02_P3.50mm_Vertical, symbol Connector:Screw_Terminal_01x02
- Q5, Q6: footprint Package_TO_SOT_THT:TO-92L_HandSolder -> Package_TO_SOT_THT:TO-92_HandSolder
Changed lines of the file:
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@@
     (property "Reference" "Q6" (id 0) (at 111.76 115.57 90))
     (property "Value" "IRF520" (id 1) (at 111.76 118.11 90))
-    (property "Footprint" "Package_TO_SOT_THT:TO-92L_HandSolder" (id 2) (at 118.11 115.57 0)
+    (property "Footprint" "Package_TO_SOT_THT:TO-92_HandSolder" (id 2) (at 118.11 115.57 0)
       (effects (font (size 1.27 1.27) italic) (justify left) hide)
     )
@@
     (pin "4")
     (pin "5")
-  )
-  (symbol (lib_id "Connector:Screw_Terminal_01x02") (at 118.11 40.64 90) (unit 1)
-    (in_bom yes) (on_board yes)
-    (property "Reference" "J7" (id 0) (at 123.19 35.56 90)
-      (effects (font (size 1.27 1.27)) (justify left))
-    )
-    (property "Value" "Screw_Terminal_01x02" (id 1) (at 124.46 38.1 90)
-      (effects (font (size 1.27 1.27)) (justify left))
-    )
-    (property "Footprint" "TerminalBlock_4Ucon:TerminalBlock_4Ucon_1x02_P3.50mm_Vertical" (id 2) (at 118.11 40.64 0)
-      (effects (font (size 1.27 1.27)) hide)
-    )
-    (property "Datasheet" "~" (id 3) (at 118.11 40.64 0)
-      (effects (font (size 1.27 1.27)) hide)
-    )
-    (pin "1")
-    (pin "2")
   )
   (symbol (lib_id "Connector:Screw_Terminal_01x02") (at 234.95 74.93 270) (unit 1)
@@
     (property "Reference" "Q5" (id 0) (at 111.76 96.52 90))
     (property "Value" "IRF520" (id 1) (at 111.76 99.06 90))
-    (property "Footprint" "Package_TO_SOT_THT:TO-92L_HandSolder" (id 2) (at 118.11 96.52 0)
+    (property "Footprint" "Package_TO_SOT_THT:TO-92_HandSolder" (id 2) (at 118.11 96.52 0)
       (effects (font (size 1.27 1.27) italic) (justify left) hide)
     )
@@
     (pin "3")
   )
-  (symbol (lib_id "mine:+8V6") (at 118.11 45.72 180) (unit 1)
-    (in_bom yes) (on_board yes) (fields_autoplaced)
-    (property "Reference" "#PWR014" (id 0) (at 118.11 41.91 0)
-      (effects (font (size 1.27 1.27)) hide)
-    )
-    (property "Value" "+8V6" (id 1) (at 118.11 50.8 0))
-    (property "Footprint" "" (id 2) (at 118.11 45.72 0)
-      (effects (font (size 1.27 1.27)) hide)
-    )
-    (property "Datasheet" "" (id 3) (at 118.11 45.72 0)
-      (effects (font (size 1.27 1.27)) hide)
-    )
-    (pin "1")
-  )
   (symbol (lib_id "Transistor_FET:BS107") (at 85.09 135.89 0) (unit 1)
     (in_bom yes) (on_board yes) (fields_autoplaced)
@@
     (pin "1")
   )
-  (symbol (lib_id "power:GND") (at 120.65 45.72 90) (unit 1)
-    (in_bom yes) (on_board yes) (fields_autoplaced)
-    (property "Reference" "#PWR015" (id 0) (at 127 45.72 0)
-      (effects (font (size 1.27 1.27)) hide)
-    )
-    (property "Value" "GND" (id 1) (at 124.46 45.7199 90)
-      (effects (font (size 1.27 1.27)) (justify right))
-    )
-    (property "Footprint" "" (id 2) (at 120.65 45.72 0)
-      (effects (font (size 1.27 1.27)) hide)
-    )
-    (property "Datasheet" "" (id 3) (at 120.65 45.72 0)
-      (effects (font (size 1.27 1.27)) hide)
-    )
-    (pin "1")
-  )
   (symbol (lib_id "power:GND") (at 184.15 52.07 0) (unit 1)
     (in_bom yes) (on_board yes) (fields_autoplaced)
@@
       (reference "#PWR013") (unit 1) (value "GND") (footprint "")
     )
-    (path "/911a3873-9972-4266-bb91-f9100ab685d2"
-      (reference "#PWR014") (unit 1) (value "+8V6") (footprint "")
-    )
-    (path "/f9d1d5de-d550-469d-ba16-03b055e1a2db"
-      (reference "#PWR015") (unit 1) (value "GND") (footprint "")
-    )
     (path "/639fda25-19c2-4900-90f9-352559cd2381"
       (reference "#PWR0101") (unit 1) (value "GND") (footprint "")
@@
       (reference "J6") (unit 1) (value "Screw_Terminal_01x02") (footprint "TerminalBlock_4Ucon:TerminalBlock_4Ucon_1x02_P3.50mm_Vertical")
     )
-    (path "/30aef055-f6a1-4cf7-bee2-a0b6411c07b3"
-      (reference "J7") (unit 1) (value "Screw_Terminal_01x02") (footprint "TerminalBlock_4Ucon:TerminalBlock_4Ucon_1x02_P3.50mm_Vertical")
-    )
     (path "/2ae5c0e2-89c9-44b0-9d9d-58442a1d2904"
       (reference "J8") (unit 1) (value "USB_A") (footprint "Connector_USB:USB_A_Molex_105057_Vertical")
@@
     )
     (path "/791fbfac-5281-4b93-9ad9-a5aba5135fdc"
-      (reference "Q5") (unit 1) (value "IRF520") (footprint "Package_TO_SOT_THT:TO-92L_HandSolder")
+      (reference "Q5") (unit 1) (value "IRF520") (footprint "Package_TO_SOT_THT:TO-92_HandSolder")
     )
     (path "/29eab021-c5d4-4a3f-bd88-e6ccee411acf"
-      (reference "Q6") (unit 1) (value "IRF520") (footprint "Package_TO_SOT_THT:TO-92L_HandSolder")
+      (reference "Q6") (unit 1) (value "IRF520") (footprint "Package_TO_SOT_THT:TO-92_HandSolder")
     )
     (path "/df93f76b-86da-45ae-87e2-4b691af12b00"
