File: pcb/system/system.kicad_sch (KiCad schematic)
At the start: 39 parts, among them J1 Raspberry_Pi_4_GPIO, J10 Conn_02x08_Odd_Even, J11 Conn_02x04_Odd_Even, J12 Conn_02x04_Odd_Even, J2 Screw_Terminal_01x02, J3 Servo_1_Header, J4 Servo_2_Header, J5 Screw_Terminal_01x02, J6 Screw_Terminal_01x02, J8 USB_A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

Commit message: updated fixed body data
Parts:
- added D5, D6: 1N746A, Diode_THT:D_DO-35_SOD27_P7.62mm_Horizontal, symbol Diode:BZV55C3V3
- added J7: Screw_Terminal_01x02, TerminalBlock_4Ucon:TerminalBlock_4Ucon_1x02_P3.50mm_Vertical, symbol Connector:Screw_Terminal_01x02
- added R10, R12: 1.2kΩ, Resistor_THT:R_Axial_DIN0204_L3.6mm_D1.6mm_P5.08mm_Horizontal, symbol pspice:R
- added R11, R9: 110Ω, Resistor_THT:R_Axial_DIN0204_L3.6mm_D1.6mm_P5.08mm_Horizontal, symbol pspice:R
Connections:
- net +8V: now also Q5.1 (G), Q6.1 (G), SW1.2 (B)
- net GND: now also D5.2 (A), D6.2 (A)
- net at R1.1, R2.1, R5.1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: now also R10.1, R12.1
- net at U1.25 (18_A4_SDA0): now also D6.1 (K), R11.2, R12.2
- net at U1.26 (19_A5_SCL0): now also D5.1 (K), R10.2, R9.2
- new net: J7.2 (Pin_2), R9.1
- new net: J7.1 (Pin_1), R11.1
- no-connect marks 123 -> 121
Other:
- moved on the sheet: C1, C2, D1, D2, D3, D4, J1, J10, J11, J12, J2, J3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
