File: pcb/system/system.kicad_sch (KiCad schematic)
At the start: 46 parts, among them J1 Raspberry_Pi_4_GPIO, J10 Conn_02x08_Odd_Even, J11 Conn_02x04_Odd_Even, J12 Conn_02x04_Odd_Even, J2 Screw_Terminal_01x02, J3 Servo_1_Header, J4 Servo_2_Header, J5 Screw_Terminal_01x02, J6 Screw_Terminal_01x02, J7 Screw_Terminal_01x02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

Commit message: updates
Parts:
- removed Q5, Q6: IRF520, Package_TO_SOT_THT:TO-92_HandSolder, symbol ze_symbols:IRF520
- removed SW1: SW_SPST, Button_Switch_THT:SW_CuK_JS202011CQN_DPDT_Straight, symbol Switch:SW_SPST
Connections:
- net +8V: now also J3.2 (Pin_2), J4.2 (Pin_2)
- net at R1.1, R10.1, R12.1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: now also U1.31 (3V3); no longer U1.33 (VIN)
Other:
- moved on the sheet: C1, C2, D1, D2, D3, D4, D5, D6, J1, J10, J11, J12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
